File: KiCad-PCB/MagSpoofTC.sch (KiCad schematic (older format))
At the start: 11 parts, among them IC1 ATTINY85-P, P1 Battery, P2 AVR ICSP, SW1 SW_PUSH, U1 TC4424

Commit message: Update version 1.1
Parts:
- C1: footprint theinventorhouse:1411(3528m)-B%2CM%2CH%2CT-TANTALUM -> theinventorhouse:CP_4x5mm; Alimentacion (none) -> 6.3v; Description (none) -> KEMET T520T107M006ATE070 CAP, TANT, POLYMER, 100UF, 6.3V, 1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; Manufacturer (none) -> Kemet; Temperatura (none) -> +85/-40
- C2: footprint theinventorhouse:1411(3528m)-B%2CM%2CH%2CT-TANTALUM -> theinventorhouse:CP_4x5mm; Alimentacion 5v -> 6.3v; Description (none) -> KEMET T520T107M006ATE070 CAP, TANT, POLYMER, 100UF, 6.3V, 1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; Manufacturer Maxim -> Kemet
- C3: footprint Capacitors_SMD:C_0603_HandSoldering -> Capacitors_ThroughHole:C_Disc_D3_P2.5; Alimentacion 5v -> 50v; Description (none) -> WALSIN 0603F104Z500CT CAP, MLCC, Y5V, 0.1UF, 50V, 0603, REEL; Manufacturer Maxim -> WALSIN
- D1: footprint LEDs:LED-0805 -> LEDs:LED-3MM; Alimentacion (none) -> 5v; Description (none) -> Led red 0805; Manufacturer (none) -> Maxim; Temperatura (none) -> +85/-40
- IC1: Alimentacion (none) -> 5v; Description (none) -> ATMEL ATTINY85-20PU Microcontrolador 8 Bits, Baja Potencia,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; Manufacturer (none) -> ATMEL; Temperatura (none) -> +85/-40
- R1: footprint Resistors_SMD:R_0603_HandSoldering -> Resistors_ThroughHole:Resistor_Horizontal_RM7mm; Alimentacion (none) -> 5v; Description (none) -> Resistor 330ohms; Temperatura (none) -> +85/-40
- U1: Alimentacion (none) -> 2.7-5v; Description (none) -> MICROCHIP TC4424CPA MOSFET Driver Lado Bajo, Alimentación:4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; Manufacturer (none) -> Microchip; Temperatura (none) -> +85/-40
Changed lines of the file:
@@
 Sheet 1 1
 Title "MagSpoof"
-Date "2016-02-22"
-Rev "1.0"
+Date "2016-07-09"
+Rev "1.1"
 Comp "Electronic Cats"
 Comment1 "Andrés Sabas"
@@
 F 1 "ATTINY85-P" H 5750 2900 40  0000 C CNN
 F 2 "Housings_DIP:DIP-8_W7.62mm_LongPads" H 5750 3300 35  0001 C CIN
-F 3 "" H 4750 3300 60  0000 C CNN
+F 3 "http://www.farnell.com/datasheets/1744708.pdf" H 4750 3300 60  0001 C CNN
+F 4 "ATMEL" H 4750 3300 60  0001 C CNN "Manufacturer"
+F 5 "+85/-40" H 4750 3300 60  0001 C CNN "Temperatura"
+F 6 "5v" H 4750 3300 60  0001 C CNN "Alimentacion"
+F 7 "ATMEL 	ATTINY85-20PU  Microcontrolador 8 Bits, Baja Potencia, Alto Rendimiento, ATtiny, 20 MHz, 8 KB, 500 Byte, 8 Pines" H 4750 3300 60  0001 C CNN "Description"
 	1    4750 3300
 	-1   0    0    -1
@@
 F 0 "D1" H 6500 3950 50  0000 C CNN
 F 1 "LED" H 6500 3750 50  0000 C CNN
-F 2 "LEDs:LED-0805" H 6500 3850 60  0001 C CNN
+F 2 "LEDs:LED-3MM" H 6500 3850 60  0001 C CNN
 F 3 "" H 6500 3850 60  0000 C CNN
+F 4 "Maxim" H 6500 3850 60  0001 C CNN "Manufacturer"
+F 5 "+85/-40" H 6500 3850 60  0001 C CNN "Temperatura"
+F 6 "5v" H 6500 3850 60  0001 C CNN "Alimentacion"
+F 7 "Led red 0805" H 6500 3850 60  0001 C CNN "Description"
 	1    6500 3850
 	0    -1   -1   0
@@
 F 0 "R1" V 6580 4350 50  0000 C CNN
 F 1 "330" V 6500 4350 50  0000 C CNN
-F 2 "Resistors_SMD:R_0603_HandSoldering" V 6430 4350 30  0001 C CNN
+F 2 "Resistors_ThroughHole:Resistor_Horizontal_RM7mm" V 6430 4350 30  0001 C CNN
 F 3 "" H 6500 4350 30  0000 C CNN
+F 4 "+85/-40" H 6500 4350 60  0001 C CNN "Temperatura"
+F 5 "5v" H 6500 4350 60  0001 C CNN "Alimentacion"
+F 6 "Resistor 330ohms" H 6500 4350 60  0001 C CNN "Description"
 	1    6500 4350
 	1    0    0    -1
@@
 F 0 "C1" H 8575 3800 50  0000 L CNN
 F 1 "100uF" H 8575 3600 50  0000 L CNN
-F 2 "theinventorhouse:1411(3528m)-B%2CM%2CH%2CT-TANTALUM" H 8588 3550 30  0001 C CNN
-F 3 "" H 8550 3700 60  0000 C CNN
+F 2 "theinventorhouse:CP_4x5mm" H 8588 3550 30  0001 C CNN
+F 3 "http://www.farnell.com/datasheets/1923743.pdf" H 8550 3700 60  0001 C CNN
+F 4 "Kemet" H 8550 3700 60  0001 C CNN "Manufacturer"
+F 5 "+85/-40" H 8550 3700 60  0001 C CNN "Temperatura"
+F 6 "6.3v" H 8550 3700 60  0001 C CNN "Alimentacion"
+F 7 "KEMET 	T520T107M006ATE070  CAP, TANT, POLYMER, 100UF, 6.3V, 1411" H 8550 3700 60  0001 C CNN "Description"
 	1    8550 3700
 	1    0    0    -1
@@
 Connection ~ 3250 3550
 $Comp
-L CP C2
-U 1 1 569FD30B
-P 5350 4400
-F 0 "C2" H 5375 4500 50  0000 L CNN
-F 1 "100uF" H 5375 4300 50  0000 L CNN
-F 2 "theinventorhouse:1411(3528m)-B%2CM%2CH%2CT-TANTALUM" H 5388 4250 30  0001 C CNN
-F 3 "" H 5350 4400 60  0000 C CNN
-F 4 "Maxim" H 5350 4400 60  0001 C CNN "Manufacturer"
-F 5 "+85/-40" H 5350 4400 60  0001 C CNN "Temperatura"
-F 6 "5v" H 5350 4400 60  0001 C CNN "Alimentacion"
-	1    5350 4400
-	1    0    0    -1
-$EndComp
-$Comp
 L C C3
 U 1 1 569FD413
@@
 F 0 "C3" H 5675 4500 50  0000 L CNN
 F 1 "0.1uF" H 5675 4300 50  0000 L CNN
-F 2 "Capacitors_SMD:C_0603_HandSoldering" H 5688 4250 30  0001 C CNN
-F 3 "" H 5650 4400 60  0000 C CNN
-F 4 "Maxim" H 5650 4400 60  0001 C CNN "Manufacturer"
+F 2 "Capacitors_ThroughHole:C_Disc_D3_P2.5" H 5688 4250 30  0001 C CNN
+F 3 "http://www.farnell.com/datasheets/2009679.pdf" H 5650 4400 60  0001 C CNN
+F 4 "WALSIN" H 5650 4400 60  0001 C CNN "Manufacturer"
 F 5 "+85/-40" H 5650 4400 60  0001 C CNN "Temperatura"
-F 6 "5v" H 5650 4400 60  0001 C CNN "Alimentacion"
+F 6 "50v" H 5650 4400 60  0001 C CNN "Alimentacion"
+F 7 "WALSIN 	0603F104Z500CT  CAP, MLCC, Y5V, 0.1UF, 50V, 0603, REEL" H 5650 4400 60  0001 C CNN "Description"
 	1    5650 4400
 	1    0    0    -1
@@
 F 1 "TC4424" H 7650 2850 60  0000 C CNN
 F 2 "Housings_DIP:DIP-8_W7.62mm_LongPads" H 7800 3200 60  0001 C CNN
-F 3 "" H 7800 3200 60  0000 C CNN
+F 3 "http://www.farnell.com/datasheets/95980.pdf" H 7800 3200 60  0001 C CNN
+F 4 "Microchip" H 7800 3200 60  0001 C CNN "Manufacturer"
+F 5 "+85/-40" H 7800 3200 60  0001 C CNN "Temperatura"
+F 6 "2.7-5v" H 7800 3200 60  0001 C CNN "Alimentacion"
+F 7 "MICROCHIP 	TC4424CPA  MOSFET Driver Lado Bajo, Alimentación:4.5-18V, Salida Pico:3A, Salida:3.5 Ohm, DIP-" H 7800 3200 60  0001 C CNN "Description"
 	1    7800 3200
 	1    0    0    -1
@@
 	8300 3250 8550 3250
 Connection ~ 8550 3250
+$Comp
+L CP C2
+U 1 1 576EF8F9
+P 5350 4400
+F 0 "C2" H 5375 4500 50  0000 L CNN
+F 1 "100uF" H 5375 4300 50  0000 L CNN
+F 2 "theinventorhouse:CP_4x5mm" H 5388 4250 30  0001 C CNN
+F 3 "http://www.farnell.com/datasheets/1923743.pdf" H 5350 4400 60  0001 C CNN
+F 4 "Kemet" H 5350 4400 60  0001 C CNN "Manufacturer"
+F 5 "+85/-40" H 5350 4400 60  0001 C CNN "Temperatura"
+F 6 "6.3v" H 5350 4400 60  0001 C CNN "Alimentacion"
+F 7 "KEMET 	T520T107M006ATE070  CAP, TANT, POLYMER, 100UF, 6.3V, 1411" H 5350 4400 60  0001 C CNN "Description"
+	1    5350 4400
+	1    0    0    -1
+$EndComp
 $EndSCHEMATC

Commit message: added BOM
Parts:
- C1, C2: Description KEMET T520T107M006ATE070 CAP, TANT, POLYMER, 100UF, 6.3V, 1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 -> (none); manf# (none) -> EEU-FC0J101
- C3: Description WALSIN 0603F104Z500CT CAP, MLCC, Y5V, 0.1UF, 50V, 0603, REEL -> (none); manf# (none) -> K104K15X7RF5TL2
- D1: symbol LED -> LED-RESCUE-MagSpoofTC; Description Led red 0805 -> (none); manf# (none) -> WP710A10QBC/D
- IC1: Description ATMEL ATTINY85-20PU Microcontrolador 8 Bits, Baja Potencia,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 -> (none); manf# (none) -> ATtiny85-20PU
- R1: Description Resistor 330ohms -> (none); manf# (none) -> ESR10EZPF3300
- U1: Description MICROCHIP TC4424CPA MOSFET Driver Lado Bajo, Alimentación:4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 -> (none); manf# (none) -> TC4424CPA
Changed lines of the file:
@@
 EESchema Schematic File Version 2
+LIBS:MagSpoofTC-rescue
 LIBS:power
 LIBS:device
@@
 LIBS:contrib
 LIBS:valves
-LIBS:theinventorhouse
 LIBS:MagSpoofTC-cache
 EELAYER 25 0
@@
 F 5 "+85/-40" H 4750 3300 60  0001 C CNN "Temperatura"
 F 6 "5v" H 4750 3300 60  0001 C CNN "Alimentacion"
-F 7 "ATMEL 	ATTINY85-20PU  Microcontrolador 8 Bits, Baja Potencia, Alto Rendimiento, ATtiny, 20 MHz, 8 KB, 500 Byte, 8 Pines" H 4750 3300 60  0001 C CNN "Description"
+F 7 "ATtiny85-20PU" H 4750 3300 60  0001 C CNN "manf#"
 	1    4750 3300
 	-1   0    0    -1
 $EndComp
 $Comp
-L LED D1
+L LED-RESCUE-MagSpoofTC D1
 U 1 1 569ED258
 P 6500 3850
@@
 F 5 "+85/-40" H 6500 3850 60  0001 C CNN "Temperatura"
 F 6 "5v" H 6500 3850 60  0001 C CNN "Alimentacion"
-F 7 "Led red 0805" H 6500 3850 60  0001 C CNN "Description"
+F 7 "WP710A10QBC/D" H 6500 3850 60  0001 C CNN "manf#"
 	1    6500 3850
 	0    -1   -1   0
@@
 F 4 "+85/-40" H 6500 4350 60  0001 C CNN "Temperatura"
 F 5 "5v" H 6500 4350 60  0001 C CNN "Alimentacion"
-F 6 "Resistor 330ohms" H 6500 4350 60  0001 C CNN "Description"
+F 6 "ESR10EZPF3300" H 6500 4350 60  0001 C CNN "manf#"
 	1    6500 4350
 	1    0    0    -1
@@
 F 5 "+85/-40" H 8550 3700 60  0001 C CNN "Temperatura"
 F 6 "6.3v" H 8550 3700 60  0001 C CNN "Alimentacion"
-F 7 "KEMET 	T520T107M006ATE070  CAP, TANT, POLYMER, 100UF, 6.3V, 1411" H 8550 3700 60  0001 C CNN "Description"
+F 7 "EEU-FC0J101" H 8550 3700 60  0001 C CNN "manf#"
 	1    8550 3700
 	1    0    0    -1
@@
 F 5 "+85/-40" H 5650 4400 60  0001 C CNN "Temperatura"
 F 6 "50v" H 5650 4400 60  0001 C CNN "Alimentacion"
-F 7 "WALSIN 	0603F104Z500CT  CAP, MLCC, Y5V, 0.1UF, 50V, 0603, REEL" H 5650 4400 60  0001 C CNN "Description"
+F 7 "K104K15X7RF5TL2" H 5650 4400 60  0001 C CNN "manf#"
 	1    5650 4400
 	1    0    0    -1
@@
 F 5 "+85/-40" H 7800 3200 60  0001 C CNN "Temperatura"
 F 6 "2.7-5v" H 7800 3200 60  0001 C CNN "Alimentacion"
-F 7 "MICROCHIP 	TC4424CPA  MOSFET Driver Lado Bajo, Alimentación:4.5-18V, Salida Pico:3A, Salida:3.5 Ohm, DIP-" H 7800 3200 60  0001 C CNN "Description"
+F 7 "TC4424CPA" H 7800 3200 60  0001 C CNN "manf#"
 	1    7800 3200
 	1    0    0    -1
@@
 F 5 "+85/-40" H 5350 4400 60  0001 C CNN "Temperatura"
 F 6 "6.3v" H 5350 4400 60  0001 C CNN "Alimentacion"
-F 7 "KEMET 	T520T107M006ATE070  CAP, TANT, POLYMER, 100UF, 6.3V, 1411" H 5350 4400 60  0001 C CNN "Description"
+F 7 "EEU-FC0J101" H 5350 4400 60  0001 C CNN "manf#"
 	1    5350 4400
 	1    0    0    -1

Commit message: fix cap 100 uF
Parts:
- C2: manf# EEU-FC0J101 -> 107KXM010M
Changed lines of the file:
@@
 F 5 "+85/-40" H 5350 4400 60  0001 C CNN "Temperatura"
 F 6 "6.3v" H 5350 4400 60  0001 C CNN "Alimentacion"
-F 7 "EEU-FC0J101" H 5350 4400 60  0001 C CNN "manf#"
+F 7 "107KXM010M" H 5350 4400 60  0001 C CNN "manf#"
 	1    5350 4400
 	1    0    0    -1

Commit message: fix cap's
Parts:
- C1: manf# EEU-FC0J101 -> 107KXM010M
- C3: manf# K104K15X7RF5TL2 -> 21RZ310-RC
Changed lines of the file:
@@
 F 5 "+85/-40" H 8550 3700 60  0001 C CNN "Temperatura"
 F 6 "6.3v" H 8550 3700 60  0001 C CNN "Alimentacion"
-F 7 "EEU-FC0J101" H 8550 3700 60  0001 C CNN "manf#"
+F 7 "107KXM010M" H 8550 3700 60  0001 C CNN "manf#"
 	1    8550 3700
 	1    0    0    -1
@@
 F 5 "+85/-40" H 5650 4400 60  0001 C CNN "Temperatura"
 F 6 "50v" H 5650 4400 60  0001 C CNN "Alimentacion"
-F 7 "K104K15X7RF5TL2" H 5650 4400 60  0001 C CNN "manf#"
+F 7 "21RZ310-RC" H 5650 4400 60  0001 C CNN "manf#"
 	1    5650 4400
 	1    0    0    -1
